File: Collier_Chien/alimentation.kicad_sch (KiCad schematic)
At the start: 21 parts, among them J1 HARVESTER, J2 SUPERCAP 5.5V, U2 BQ25570

Commit message: Restaure la feuille BQ25570 EDU RAK a identique
Parts:
- removed C1: 4.7uF / 10V, Capacitor_SMD:C_0603_1608Metric, symbol Collier:C
- removed C2, C5, C7: 100nF / 10V, Capacitor_SMD:C_0603_1608Metric, symbol Collier:C
- removed C3: 10nF / faible fuite, Capacitor_SMD:C_0603_1608Metric, symbol Collier:C
- removed C4, C6: 22uF / 10V, Capacitor_SMD:C_0603_1608Metric, symbol Collier:C
- removed J1: HARVESTER, Connector_PinHeader_2.54mm:PinHeader_1x02_P2.54mm_Vertical, symbol Collier:Conn_01x02_Pin
- removed J2: SUPERCAP 5.5V, Connector_PinHeader_2.54mm:PinHeader_1x02_P2.54mm_Vertical, symbol Collier:Conn_01x02_Pin
- removed L1: 22uH / Isat >= 0.3A, symbol Collier:L
- removed L2: 10uH / Isat >= 0.3A, symbol Collier:L
- removed R1: 8.66M, Resistor_SMD:R_0603_1608Metric, symbol Collier:R
- removed R2: 7.15M, Resistor_SMD:R_0603_1608Metric, symbol Collier:R
- removed R3: 0.681M, Resistor_SMD:R_0603_1608Metric, symbol Collier:R
- removed R4, R6: 8.25M, Resistor_SMD:R_0603_1608Metric, symbol Collier:R
- removed R5: 4.12M, Resistor_SMD:R_0603_1608Metric, symbol Collier:R
- removed R7: 4.75M, Resistor_SMD:R_0603_1608Metric, symbol Collier:R
- removed R8: 1M, Resistor_SMD:R_0603_1608Metric, symbol Collier:R
- removed R9: 2M, Resistor_SMD:R_0603_1608Metric, symbol Collier:R
- removed U2: BQ25570, Package_DFN_QFN:QFN-20-1EP_3.5x3.5mm_P0.5mm_EP2x2mm, symbol Collier:BQ25570
- added C1, CBYP1, CIN1: 100nF, Capacitor_SMD:C_0603_1608Metric, symbol Device:C
- added C22: 100uF, Capacitor_SMD:C_0603_1608Metric, symbol Device:C
- added CIN2: 4.7uF, Capacitor_SMD:C_0603_1608Metric, symbol Device:C
- added COUT1, CSTOR1: 22uF, Capacitor_SMD:C_0603_1608Metric, symbol Device:C
- added CREF1: 10nF, Capacitor_SMD:C_0603_1608Metric, symbol Device:C
- added J10: P-MFC, TerminalBlock_Phoenix:TerminalBlock_Phoenix_MKDS-3-2-5.08_1x02_P5.08mm_Horizontal, symbol Connector:Screw_Terminal_01x02
- added J19: Conn_01x02_Socket, Connector_PinSocket_2.54mm:PinSocket_1x02_P2.54mm_Vertical, symbol Connector:Conn_01x02_Socket
- added J3, J4: Conn_01x02_Pin, Connector_PinHeader_2.54mm:PinHeader_1x02_P2.54mm_Vertical, symbol Connector:Conn_01x02_Pin
- added LBOOST1: 22uH, LPS4018-223MRC:IND_LPS4018-223MRC, symbol Device:L
- added LBUCK1: 10uH, Inductor_SMD:L_1008_2520Metric, symbol Device:L
- added ROK1: 4.22M, Resistor_SMD:R_0603_1608Metric, symbol Device:R
- added ROK1B1, ROK2B1, ROK3B1, ROUT1B1, ROUT2B1, ROV1B1, ROV2B1: R, Resistor_SMD:R_0603_1608Metric, symbol Device:R
- added ROK2: 7.87M, Resistor_SMD:R_0603_1608Metric, symbol Device:R
- added ROK3: 1.1M, Resistor_SMD:R_0603_1608Metric, symbol Device:R
- added ROUT1: 4.64M, Resistor_SMD:R_0603_1608Metric, symbol Device:R
- added ROUT2: 8.25M, Resistor_SMD:R_0603_1608Metric, symbol Device:R
- added ROV1: 7.15M, Resistor_SMD:R_0603_1608Metric, symbol Device:R
- added ROV2: 8.66M, Resistor_SMD:R_0603_1608Metric, symbol Device:R
- added U2: BQ25570, Package_DFN_QFN:QFN-20-1EP_3.5x3.5mm_P0.5mm_EP2x2mm, symbol Battery_Management:BQ25570
Connections:
- net GND: now also C1.2, C22.2, CBYP1.2, CIN1.2, CIN2.2, COUT1.1, CREF1.2, CSTOR1.2, J10.2 (Pin_2), J19.1 (Pin_1), ROK1.2, ROK1B1.2, ROUT1.2, ROUT1B1.2, ROV1.2, ROV1B1.2, U2.1 (VSS), U2.15 (VSS), U2.17 (VSS), U2.21 (VSS), U2.9 (VSS)
- net VRDIV: now also ROK3.1, ROK3B1.1, ROUT2.1, ROUT2B1.1, ROV2.1, ROV2B1.1, U2.8 (VRDIV)
- new net: CIN1.1, CIN2.1, J4.2 (Pin_2), LBOOST1.1, U2.2 (VIN_DC)
- new net: ROV1.1, ROV1B1.1, ROV2.2, ROV2B1.2, U2.7 (VBAT_OV)
- new net: ROK2.1, ROK2B1.1, ROK3.2, ROK3B1.2, U2.10 (OK_HYST)
- new net: ROK1.1, ROK1B1.1, ROK2.2, ROK2B1.2, U2.11 (OK_PROG)
- new net: C1.1, C22.1, U2.18 (VBAT)
- new net: J10.1 (Pin_1), J4.1 (Pin_1)
- new net: CREF1.1, U2.4 (VREF_SAMP)
- new net: ROUT1.1, ROUT1B1.1, ROUT2.2, ROUT2B1.2, U2.12 (VOUT_SET)
- new net: COUT1.2, J3.1 (Pin_1), LBUCK1.2, U2.14 (VOUT)
- new net: LBUCK1.1, U2.16 (LBUCK)
- new net: LBOOST1.2, U2.20 (LBOOST)
- new net 'EN: U2.5 (~{EN})
- new net PWR: J3.2 (Pin_2)
- new net VBAT_OK: U2.13 (VBAT_OK)
- new net VOUT_EN: CBYP1.1, CSTOR1.1, J19.2 (Pin_2), U2.19 (VSTOR), U2.3 (VOC_SAMP), U2.6 (VOUT_EN)
Other:
- note removed: "01 RECUPERATION D'ENERGIE ET STOCKAGE"
- note removed: "MPPT = 80% (VOC_SAMP a VSTOR) Entree DC : 0.6V min au demarrage ; 5.1V max en service. J2 : supercondensateur externe >= 5.5V, capacite a dimensionner. VBAT_OK commande le buck ; arret ~3.63V / reprise ~3.83V. VBAT_OV ~4.01V ; VOUT ~3.31V nominal. Pont R8/R9 : adaptation de VBAT_OK vers le MCU."
- note removed: "Seuils de stockage et sortie - resistances 1%"
- company: Collier chien / Amira -> DD
- title: Alimentation / BQ25570 -> Edu_RAK_2026
