File: Collier_Chien/accelerometre.kicad_sch (KiCad schematic)
At the start: 6 parts, among them U3 LIS2HH12

Commit message: Restaure la feuille BQ25570 EDU RAK a identique
Connections:
- net 3V3 renamed PWR
