File: Collier_Chien/collier_chien.kicad_sch (KiCad schematic)
At the start: 0 parts

Commit message: Restaure la feuille BQ25570 EDU RAK a identique
Other:
- note added: "Alimentation regulee ~3.36V (reglage EDU RAK). Mesure par I2C et reveil par interruption. Stockage : supercondensateur externe ; source de recuperation a choisir. Cette revision contient uniquement le schema et les controles electriques. Autonomie, transitoires radio et dimensionnement de la source a valider avant PCB."
- note removed: "Alimentation regulee 3.31V. Mesure par I2C et reveil par interruption. Stockage : supercondensateur externe ; source de recuperation a choisir. Cette revision contient uniquement le schema et les controles electriques. Autonomie, transitoires radio et dimensionnement de la source a valider avant PCB."
