File: Collier_Chien/rak3172.kicad_sch (KiCad schematic)
At the start: 10 parts, among them J3 ANTENNE 868MHz / 50 ohms, J4 UART2 / RUI3, J5 SWD, SW1 RESET, U1 RAK3172(H) / EU868

Commit message: Restaure la feuille BQ25570 EDU RAK a identique
Parts:
- added R8: 1M, Resistor_SMD:R_0603_1608Metric, symbol Collier:R
- added R9: 2M, Resistor_SMD:R_0603_1608Metric, symbol Collier:R
- renumbered J3 to J20, J4 to J21, J5 to J22
Connections:
- net GND: now also R9.2
- net VBAT_OK_3V3: now also R8.2, R9.1
- net 3V3 renamed PWR
- new net VBAT_OK: R8.1
Other:
- note added: "Alimentation via le cavalier J3 de la feuille BQ originale."

Commit message: Personnalise le depot du collier et verifie le schema avec antenne 868 MHz
Parts:
- added AE1: Antenne generique 868 MHz, symbol Collier:Antenna_868MHz
Connections:
- net RF: now also AE1.1 (A)
- net GND renamed 'EN
Other:
- note added: "AE1 : antenne externe indicative / 50 ohms. Frequence cible 868 MHz ; modele physique a choisir."
- note added: "BQ actif : EN relie a GND par le label global de la feuille originale."
