File: VeillePorte/alimentation.kicad_sch (KiCad schematic)
At the start: 29 parts, among them J10 P-MFC, J19 Conn_01x02_Socket, J3 Conn_01x02_Pin, J4 Conn_01x02_Pin, U2 BQ25570

Commit message: Regle le BQ25570 pour supercapacite 4V et structure la feuille RAK
Parts:
- ROK1, ROK2: Tolerance (none) -> 0.1%
- ROK3: value 1.1M -> 464k; Tolerance (none) -> 0.1%
- ROUT1: value 4.64M -> 4.99M; Tolerance (none) -> 0.1%
- ROUT2: value 8.25M -> 7.87M; Tolerance (none) -> 0.1%
- ROV1: value 7.15M -> 6.19M; Tolerance (none) -> 0.1%
- ROV2: value 8.66M -> 6.81M; Tolerance (none) -> 0.1%
Connections:
- net VBAT_OK: now also U2.6 (VOUT_EN)
- net VOUT_EN: no longer names the net of CBYP1.1, CSTOR1.1, J19.2 (Pin_2), U2.19 (VSTOR), U2.3 (VOC_SAMP)
- net VOUT_EN: no longer U2.6 (VOUT_EN)
Other:
- note added: "SUPERCAPA 4V MAX : OV ~3.812V ; OK bas ~3.467V / haut ~3.600V. Sortie ~3.118V ; resistances de seuil 0.1%. VBAT_OK commande VOUT_EN : arret du buck si energie insuffisante. Options NC et C22 conservees ; stockage et pointes a verifier sur banc."
- title: Edu_RAK_2026 -> VeillePorte - BQ25570 / supercapacite 4 V
