File: VeillePorte/rak3172.kicad_sch (KiCad schematic)
At the start: 13 parts, among them J20 ANTENNE 868MHz / 50 ohms, J21 UART2 / RUI3, J22 SWD, SW1 RESET, U1 RAK3172(H) / EU868

Commit message: Remplace le LIS2HH12 par le raccordement IR VL53L4CD Pololu 3692
Connections:
- net IR_XSHUT: now reaches U1.30 (PB5)
- net ACC_INT1 renamed IR_INT
- no-connect marks 15 -> 14
Other:
- note added: "UART : adaptateur logique 3.3V ; TX adaptateur vers RX module. SWD : reference tension seulement, eviter deux alimentations simultanees. BOOT0 maintenu bas ; RUI3 se programme par UART2. PA11/PA12 : I2C2 ; PA1 : interruption IR adaptee. PB5 : XSHUT en drain ouvert (bas ou haute impedance). PA0 : etat du stockage via pont diviseur. Verifier les cretes TX et la tenue du 3V3 sur banc. RF : liaison 5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"
- note removed: "UART : adaptateur logique 3.3V ; TX adaptateur vers RX module. SWD : reference tension seulement, eviter deux alimentations simultanees. BOOT0 maintenu bas ; RUI3 se programme par UART2. PA11/PA12 : I2C2 ; PA1 : interruption accelerometre. PA0 : etat du stockage via pont diviseur. Verifier les cretes TX et la tenue du 3V3 sur banc. RF : liaison 50 ohms courte et plan de masse lors du futur PCB."

Commit message: Regle le BQ25570 pour supercapacite 4V et structure la feuille RAK
Parts:
- R9: value 2M -> 3.3M
Other:
- note added: "ALIMENTATION ET DECOUPLAGE"
- note added: "Alimentation ~3.118V via J3 ; buck commande par VBAT_OK."
- note added: "BOOT ET RESET"
- note added: "ETAT DU STOCKAGE"
- note added: "RADIO ET ANTENNE 868 MHz"
- note added: "RAK3172 - TRAITEMENT"
- note added: "UART / SWD"
- note added: "UART : adaptateur logique 3.3V ; TX adaptateur vers RX module. SWD : reference tension seulement, eviter deux alimentations simultanees. BOOT0 maintenu bas ; RUI3 se programme par UART2. PA11/PA12 : I2C2 ; PA1 : interruption IR directe 2.8V. PB5 : XSHUT en drain ouvert (bas ou haute impedance). PA0 : etat du stockage via pont diviseur. Verifier les cretes TX et la tenue du 3V3 sur banc. RF : liai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"
- note removed: "Alimentation via le cavalier J3 de la feuille BQ originale."
- note removed: "UART : adaptateur logique 3.3V ; TX adaptateur vers RX module. SWD : reference tension seulement, eviter deux alimentations simultanees. BOOT0 maintenu bas ; RUI3 se programme par UART2. PA11/PA12 : I2C2 ; PA1 : interruption IR adaptee. PB5 : XSHUT en drain ouvert (bas ou haute impedance). PA0 : etat du stockage via pont diviseur. Verifier les cretes TX et la tenue du 3V3 sur banc. RF : liaison 5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"
