File: VeillePorte/veilleporte_complet.kicad_sch (KiCad schematic)
At the start: 45 parts, among them J10 P-MFC, J19 Conn_01x02_Socket, J20 ANTENNE 868MHz / 50 ohms, J21 UART2 / RUI3, J22 SWD, J23 CABLE MODULE VL53L4CD, J3 Conn_01x02_Pin, J4 Conn_01x02_Pin, SW1 RESET, U1 RAK3172(H) / EU868, U2 BQ25570

Commit message: Lie l antenne IFA a KiCad
Parts:
- AE1: value Antenne generique 868 MHz -> Antenne IFA imprimée 868 MHz; footprint (none) -> VeillePorte_Antennes:IFA_868_CST_30x20_PisteFine
Connections:
- net RF is gone; now on net GND: AE1.1 (A), J20.1 (In), U1.12 (RF)
- net GND: now also AE1.2 (GND)

Commit message: Ajoute adaptation RF 868 MHz avec shunts DNP
Parts:
- removed J20: ANTENNE 868MHz / 50 ohms, Connector_Coaxial:U.FL_Hirose_U.FL-R-SMT-1_Vertical, symbol VeillePorte:Conn_Coaxial
- added C6: DNP, Capacitor_SMD:C_0603_1608Metric, symbol Device:C
- added L1: DNP, Inductor_SMD:L_0603_1608Metric, symbol Device:L
- added R12: 0R, Resistor_SMD:R_0603_1608Metric, symbol VeillePorte:R
Connections:
- net GND: now also C6.2, L1.2; no longer AE1.1 (A), U1.12 (RF)
- new net RF_ANT: AE1.1 (A), L1.1, R12.2
- new net RF_SRC: C6.1, R12.1, U1.12 (RF)
